File: hardware/pcb/microsd.kicad_sch (KiCad schematic)
At the start: 8 parts, among them U700 W25Q128JVP

Commit message: - PCB r0.3 routed, need to finalize
Parts:
- removed C700: 18pF/DNP, Capacitor_SMD:C_0201_0603Metric, symbol Device:C
Changed lines of the file:
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@@
   (junction (at 134.62 120.65) (diameter 0.9144) (color 0 0 0 0))
   (junction (at 134.62 134.62) (diameter 0.9144) (color 0 0 0 0))
-  (junction (at 149.86 73.66) (diameter 0.9144) (color 0 0 0 0))
   (junction (at 149.86 120.65) (diameter 0.9144) (color 0 0 0 0))
   (junction (at 149.86 147.32) (diameter 0.9144) (color 0 0 0 0))
@@
     (stroke (width 0) (type solid) (color 0 0 0 0))
   )
-  (wire (pts (xy 149.86 86.36) (xy 149.86 73.66))
-    (stroke (width 0) (type solid) (color 0 0 0 0))
-  )
-  (wire (pts (xy 149.86 93.98) (xy 149.86 96.52))
-    (stroke (width 0) (type solid) (color 0 0 0 0))
-  )
   (wire (pts (xy 149.86 127) (xy 149.86 120.65))
     (stroke (width 0) (type solid) (color 0 0 0 0))
@@
     (pin "1")
   )
-  (symbol (lib_id "power:GND") (at 149.86 96.52 0) (unit 1)
-    (in_bom yes) (on_board yes)
-    (property "Reference" "#PWR0201" (id 0) (at 149.86 102.87 0)
-      (effects (font (size 1.27 1.27)) hide)
-    )
-    (property "Value" "GND" (id 1) (at 149.987 100.9142 0))
-    (property "Footprint" "" (id 2) (at 149.86 96.52 0)
-      (effects (font (size 1.27 1.27)) hide)
-    )
-    (property "Datasheet" "" (id 3) (at 149.86 96.52 0)
-      (effects (font (size 1.27 1.27)) hide)
-    )
-    (pin "1")
-  )
   (symbol (lib_id "power:GND") (at 149.86 147.32 0) (unit 1)
     (in_bom yes) (on_board yes)
@@
       (effects (font (size 1.27 1.27)) hide)
     )
-    (pin "1")
-    (pin "2")
-  )
-  (symbol (lib_id "Device:C") (at 149.86 90.17 0) (unit 1)
-    (in_bom yes) (on_board yes)
-    (property "Reference" "C700" (id 0) (at 152.781 89.002 0)
-      (effects (font (size 1.27 1.27)) (justify left))
-    )
-    (property "Value" "18pF/DNP" (id 1) (at 152.781 91.313 0)
-      (effects (font (size 1.27 1.27)) (justify left))
-    )
-    (property "Footprint" "Capacitor_SMD:C_0201_0603Metric" (id 2) (at 150.8252 93.98 0)
-      (effects (font (size 1.27 1.27)) hide)
-    )
-    (property "Datasheet" "~" (id 3) (at 149.86 90.17 0)
-      (effects (font (size 1.27 1.27)) hide)
-    )

Commit message: - PCB layout finished for r0p3
Parts:
- renumbered MICRO_SD700 to CARD700
Changed lines of the file:
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@@
   (symbol (lib_id "symbols:MICRO_SD(TFC-WPAPR-08)") (at 170.18 76.2 0) (unit 1)
     (in_bom yes) (on_board yes)
-    (property "Reference" "MICRO_SD700" (id 0) (at 178.511 73.584 0)
+    (property "Reference" "CARD700" (id 0) (at 178.511 73.584 0)
       (effects (font (size 1.524 1.524)) (justify left))
     )
