File: hardware/pcb/ram.kicad_sch (KiCad schematic)
At the start: 20 parts, among them U300 IS66WVC4M16-ALL, U301 MT48H16M32LFB5-6 or IS42VM321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, U302 74LVC1G126, U303 IS66WVC4M16-ALL, U304 74LVC1G126

Commit message: - Working on pcb layout
Connections:
- net CRAM_CEN renamed CRAMA_CEN
Changed lines of the file:
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@@
     )
   )
-  (global_label "CRAM_CEN" (shape input) (at 106.68 38.1 180)
+  (global_label "CRAMA_CEN" (shape input) (at 106.68 38.1 180)
     (effects (font (size 1.27 1.27)) (justify right))
-    (property "Intersheet References" "${INTERSHEET_REFS}" (id 0) (at -88.9 -58.42 0)
-      (effects (font (size 1.27 1.27)) hide)
+    (property "Intersheet References" "${INTERSHEET_REFS}" (id 0) (at 91.8572 38.0206 0)
+      (effects (font (size 1.27 1.27)) (justify right) hide)
     )
   )
