File: hardware/pcb/usb.kicad_sch (KiCad schematic)
At the start: 55 parts, among them J800 USB_C_Receptacle, U800 USBLC6-2P6, U801 FUSB302UCX, U802 CBTL08GP053, U803 TC358777, X800 19.2MHz

Commit message: - Working on pcb layout
Parts:
- removed C823, C824, C825, C826, C829, C830, C831, C832, C833, C834, C835, C836: 100nF, Capacitor_SMD:C_0201_0603Metric, symbol Device:C
Connections:
- net +1V8 is gone; now on net +3V3: C817.1, U802.E4 (VDDIO), U802.H3 (VDDIO), U802.J5 (SW_EN)
- net I2C1_SCL is gone; now on net I2C3_SDA: U802.J4 (I2C_CLK)
- net I2C1_SDA is gone; now on net I2C3_SCL: U802.H4 (I2C_SDA)
- net GND: now also U802.B1 (IP5-), U802.C1 (IP5+), U802.H1 (IP2+), U802.J1 (IP2-)
- net TYPEC_RX1N: now also U802.J6 (OP1-)
- net TYPEC_RX1P: now also U802.H6 (OP1+)
- net TYPEC_RX2N: now also U802.E6 (OP2-)
- net TYPEC_RX2P: now also U802.D6 (OP2+)
- net TYPEC_TX1N: now also U802.F6 (OP3-)
- net TYPEC_TX1P: now also U802.G6 (OP3+)
- net TYPEC_TX2N: now also U802.B6 (OP4-)
- net TYPEC_TX2P: now also U802.C6 (OP4+)
- no-connect marks 3 -> 7

Commit message: - PCB r0.3 routed, need to finalize
Parts:
- removed C819, C820: 100nF, Capacitor_SMD:C_0201_0603Metric, symbol Device:C
- removed L801: 300R, Inductor_SMD:L_0603_1608Metric, symbol Device:L
- removed R802: 10K, Capacitor_SMD:C_0402_1005Metric, symbol Device:R
Connections:
- net +1V8_DP: now also U803.F7 (DISABLE_ASSR)
- net GND: now also J800.S1 (SHIELD)
- net at U803.K3 (DP_M0): now also U802.G1 (IP3-)
- net at U802.F1 (IP3+): now also U803.J3 (DP_P0)
- net VBUS_IN: now reaches J800.A4 (VBUS), J800.A9 (VBUS), J800.B4 (VBUS), J800.B9 (VBUS), L802.2, U800.5 (VBUS), U801.A2 (VBUS)

Commit message: - PCB layout finished for r0p3
Parts:
- removed U801: FUSB302UCX, Package_BGA:WLP-9_1.448x1.468mm_Layout3x3_P0.4mm_Ball0.27mm_Pad0.25mm, symbol symbols:FUSB302UCX
- added U801: FUSB302BMPX, Package_DFN_QFN:WQFN-14-1EP_2.5x2.5mm_P0.5mm_EP1.45x1.45mm, symbol Interface_USB:FUSB302BMPX
Connections:
- net +3V3: now also U801.12 (VCONN), U801.13 (VCONN), U801.3 (VDD), U801.4 (VDD)
- net GND: now also U801.15 (GND), U801.8 (GND), U801.9 (GND)
- net I2C3_SCL: now also U801.6 (SCL)
- net I2C3_SDA: now also U801.7 (SDA)
- net VBUS_IN: now also U801.2 (VBUS)
- net DP_P0: now reaches U802.F1 (IP3+), U803.J3 (DP_P0)
- net DP_N0: now reaches U802.G1 (IP3-), U803.K3 (DP_M0)
- net DP_AUXP: now reaches C827.1, U803.J10 (DP_AUXP)
- net at J800.B5 (CC2): now also U801.1 (CC2), U801.14 (CC2)
- net at J800.A5 (CC1): now also U801.10 (CC1), U801.11 (CC1)
- net DP_P1: now reaches C821.1, U803.J5 (DP_P1)
- net DP_N1: now reaches C822.1, U803.K5 (DP_M1)
- net DP_AUXN: now reaches C828.1, U803.K10 (DP_AUXM)
Other:
- moved on the sheet: C821, C822, C827, C828

Commit message: - PCB: prepare for r0p4
Parts:
- removed C804: 100nF, Capacitor_SMD:C_0201_0603Metric, symbol Device:C
- removed L807: 120R, Inductor_SMD:L_0402_1005Metric, symbol Device:L
- removed U803: TC358777, footprint:BGA-80_10x10_7.0x7.0mm, symbol symbols:TC358777
- added U803: SN65DSI86, footprint:BGA-64_9x9_5.0x5.0mm, symbol symbols:SN65DSI86
- C800: value 470nF -> DNP/470nF
- C814: value 1uF -> 10uF
- C815, C816: value 100nF -> 10nF
- R800: value 10K -> DNP/10K
- R801: value 3K/1% -> 51K/1%
- X800: value 19.2MHz -> DNP/19.2MHz
Connections:
- net +1V2_DP: no longer L805.1
- net +1V8_DP: now also L803.1, L805.1; no longer L803.2
- net DP_AUXN: now also U803.H9 (AUXN)
- net DP_AUXP: now also U803.H8 (AUXP)
- net DP_HPD: now also R801.2
- net DP_N0: now also U803.F9 (ML0N)
- net DP_N1: now also U803.E9 (ML1N)
- net DP_P0: now also U803.F8 (ML0P)
- net DP_P1: now also U803.E8 (ML1P)
- net DP_RST: now also U803.B1 (EN)
- net GND: now also U803.A1 (ADDR), U803.A8 (GND), U803.D8 (GND), U803.E4 (GND), U803.E5 (GND), U803.F4 (GND), U803.F5 (GND), U803.F6 (GND), U803.G8 (GND)
- net I2C4_SCL: now also U803.H1 (SCL)
- net I2C4_SDA: now also U803.J1 (SDA)
- net MIPI_CKN: now also U803.J5 (DACN)
- net MIPI_CKP: now also U803.H5 (DACP)
- net MIPI_D0N: now also U803.J3 (DA0N)
- net MIPI_D0P: now also U803.H3 (DA0P)
- net MIPI_D1N: now also U803.J4 (DA1N)
- net MIPI_D1P: now also U803.H4 (DA1P)
- net at C801.1, C802.1, C803.1: now also L803.2, U803.A2 (VCCIO), U803.B6 (VCCIO); no longer L803.1
- net at C805.1, C806.1, C807.1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: now also U803.D5 (VCC), U803.D6 (VCC), U803.J2 (VCC), U803.J9 (VCC)
- net at C808.1, C810.1, L805.2: now also U803.D9 (VPLL)
- net at C814.1, C815.1, C816.1: now also C811.1, C812.1, C813.1, L806.2, U803.A9 (VCCA), U803.B2 (VCCA), U803.E6 (VCCA), U803.G9 (VCCA), U803.H2 (VCCA)
- net at R801.1: now also U803.J8 (HPD)
- net at X800.3 (OUT): now also U803.A7 (REFCLK)
- no-connect marks 7 -> 26
Other:
- moved on the sheet: C800, C801, C802, C803, C805, C806, C807, C808, C810, C811, C812, C813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

Commit message: - pcb: r0p4, update to KiCAD 6.0
Parts:
- removed L806: 120R, Inductor_SMD:L_0402_1005Metric, symbol Device:L
- removed R801: 51K/1%, Capacitor_SMD:C_0402_1005Metric, symbol Device:R
- added C804: 470nF, Capacitor_SMD:C_0201_0603Metric, symbol Device:C
- added R802: 0/DNP, Capacitor_SMD:C_0402_1005Metric, symbol Device:R
Connections:
- net +1V8_DP: no longer C800.2, R800.1, X800.4 (Vdd)
- net GND: now also C804.1, R802.2
- net DP_VCCIO: now reaches C801.1, C802.1, C803.1, L803.2, U803.A2 (VCCIO), U803.B6 (VCCIO)
- net DP_VCCIO: now also C800.2, R800.1, X800.4 (Vdd)
- net DP_VCC: now reaches C805.1, C806.1, C807.1, L804.2, U803.D5 (VCC), U803.D6 (VCC), U803.J2 (VCC), U803.J9 (VCC)
- net DP_VCC: now also C811.1, C812.1, C813.1, C814.1, C815.1, C816.1, U803.A9 (VCCA), U803.B2 (VCCA), U803.E6 (VCCA), U803.G9 (VCCA), U803.H2 (VCCA)
- net DP_VPLL: now reaches C808.1, C810.1, L805.2, U803.D9 (VPLL)
- net at U803.A7 (REFCLK), X800.3 (OUT): now also R802.1
- net DP_RST: no longer names the net of U803.B1 (EN)
- net DP_RST: now also C804.2
- no-connect marks 26 -> 27
Other:
- note added: "HPD Disabled"
